File: MEMS_BMI/MEMS_BMI.sch (EAGLE design)
At the start: 85 parts, among them J1 2x3p-2.54, J2 HR911105A, J5 2X10P-2.54, K1 botton, K2 B3U-1000P, Q1 CSM-7X-DU, U1 AMS1117-3.3V, Y1 25MHZ

Commit message: intan added, BMI-V2
Parts:
- removed C10, C12, C13, C8: 104, 1-intan:CAP-(0603)
- removed HDMI-1: MICRO-HDMI, 1-intan:MICRO-HDMI
- removed J5: 2X10P-2.54, Seeed-OPL-Connector:DIP-BLACK-FEMALE-HEADER(2X10P-2.54)-2.54
- removed K2: B3U-1000P, 1-intan:SMD-BUTTON
- removed Q1: CSM-7X-DU, crystal:CSM-7X-DU
- added C18: 10n, 1-intan:CAP-(0603)
- added C32: 100n, 1-intan:CAP-(0603)
- added J3: 3P-2.54, Seeed-OPL-Connector:DIP-WHITE-MALE-HEADER-VERT(3P-2.54)
- added R34, R35, R36: 100, 1-intan:RES-(0603)
- added U$3: PROBE, 1-intan:PROBE
- added U2: RHD2216_QFN, RHD2000:RHD2216_QFN
- added Y2: 30MHZ, Seeed-OPL-Crystal-Oscillator:SMD-CRYSTAL-30MHZ-10PF-10PPM-60R(4P-3.2X2.5MM)
- R5, R6: value 22R -> 0
Connections:
- removed net N$2: R5.1, USB1.DM
- removed net N$29: K2.2, U$1.PB0
- removed net N$3: R6.1, USB1.DP
- removed net PA11/USB_DM: R5.2, U$1.PA11
- removed net PA12/USB_DP: R6.2, U$1.PA12
- new net CH0: U$3.P$16, U2.IN0+
- new net CH1: U$3.P$15, U2.IN1+
- new net CH12: U$3.P$4, U2.IN12+
- new net CH13: U$3.P$3, U2.IN13+
- new net CH14: U$3.P$2, U2.IN14+
- new net CH15: U$3.P$1, U2.IN15+
- new net CH2: U$3.P$14, U2.IN2+
- new net CH3: U$3.P$13, U2.IN3+
- new net CH4: U$3.P$12, U2.IN4+
- new net N$30: C18.2, U2.ADC_REF
- new net N$36: J3.P$3, U2.IN0-, U2.IN1-, U2.IN10-, U2.IN11-, U2.IN12-, U2.IN13-, U2.IN14-, U2.IN15-, U2.IN2-, U2.IN3-, U2.IN4-, U2.IN5-, U2.IN6-, U2.IN7-, U2.IN8-, U2.IN9-
- new net N$37: U$3.P$11, U2.IN5+
- new net N$38: U$3.P$10, U2.IN6+
- new net N$39: U$3.P$9, U2.IN7+
- new net N$40: U$3.P$8, U2.IN8+
- new net N$41: U$3.P$7, U2.IN9+
- new net N$42: U$3.P$6, U2.IN10+
- new net N$43: U$3.P$5, U2.IN11+
- net +3V3: no longer C10.1, C12.1, C13.1, C8.1, J5.11, J5.12, J5.13, J5.14, J5.15
- net CLK+: now also R35.2, U2.SCLK+; no longer HDMI-1.TX1_P
- net CLK-: now also R35.1, U2.SCLK-; no longer HDMI-1.TX1_N
- net CS+: now also R34.2, U2.!CS!+; no longer HDMI-1.TX2_P
- net CS-: now also R34.1, U2.!CS!-; no longer HDMI-1.TX2_N
- net DVCC: now also C32.2, R5.1, R5.2, U2.AUXIN1, U2.AUXIN2, U2.AUXIN3, U2.LVDS_EN, U2.VDD1, U2.VDD2, U2.VDD3; no longer HDMI-1.+5V
- net GND: now also C18.1, C32.1, J3.P$1, J3.P$2, R6.1, R6.2, U2.CTR, U2.GND0, U2.GND1, U2.GND2, U2.GND3, U2.GND4, U2.VESD; no longer C10.2, C12.2, C13.2, C8.2, HDMI-1.GND@1, HDMI-1.GND@2, HDMI-1.GND@3, HDMI-1.GND@4, HDMI-1.GND@5, HDMI-1.GND@6, HDMI-1.GND@7, HDMI-1.GND@8, HDMI-1.GND@9, J5.10, J5.5, J5.6, J5.7, J5.8, J5.9, K2.1
- net MISO+: now also U2.MISO+; no longer HDMI-1.TX0_P
- net MISO-: now also U2.MISO-; no longer HDMI-1.TX0_N
- net MOSI+: now also R36.2, U2.MOSI+; no longer HDMI-1.CLK_P
- net MOSI-: now also R36.1, U2.MOSI-; no longer HDMI-1.CLK_N
- net N$19: now also Y1.4; no longer Y1.1
- net N$27: now also Y1.2; no longer Y1.3
- net OSC_IN: now also Y2.2; no longer Q1.2
- net OSC_OUT: now also Y2.4; no longer Q1.1
- net SPI2_CLK: no longer J5.2
- net SPI2_CS: no longer J5.1
- net SPI2_MISO: no longer J5.3
- net SPI2_MOSI: no longer J5.4
- net W5500_CLK: no longer J5.19
- net W5500_CS: no longer J5.20
- net W5500_MISO: no longer J5.18
- net W5500_MOSI: no longer J5.17
- net W5500_RST: no longer J5.16
Other:
- note added: "intan"
- note added: "mcu"
